File: mosfet.kicad_sch (KiCad schematic)
At the start: 60 parts, among them J17 Screw_Terminal_01x02, J18 Screw_Terminal_01x02, J19 Screw_Terminal_01x02, J20 Screw_Terminal_01x02, J21 Screw_Terminal_01x02, J22 Screw_Terminal_01x02, J23 Screw_Terminal_01x02, J24 Screw_Terminal_01x02, J25 Screw_Terminal_01x02, J26 Screw_Terminal_01x02, J27 Screw_Terminal_01x02, J28 Screw_Terminal_01x02, J29 Screw_Terminal_01x02, J30 Screw_Terminal_01x02, Q15 IRLZ44N, Q16 IRLZ44N, Q17 IRLZ44N, Q18 IRLZ44N, Q19 IRLZ44N, Q20 IRLZ44N, Q21 IRLZ44N, Q22 IRLZ44N, Q23 IRLZ44N, Q24 IRLZ44N, Q25 IRLZ44N, Q26 IRLZ44N, Q27 IRLZ44N, Q28 IRLZ44N

Commit message: Switched the diodes on the fan to Schottkys and added a Schottky to input of power regulator
Parts:
- removed D10, D11, D12, D9: 1N4007, Diode_THT:D_DO-41_SOD81_P10.16mm_Horizontal, symbol Diode:1N4007
- added D10, D11, D12, D9: 1N5819, Diode_THT:D_DO-41_SOD81_P10.16mm_Horizontal, symbol Diode:1N5819
Connections:
- net +12V: now also D10.1 (K), D11.1 (K), D12.1 (K), D9.1 (K)
- net at J23.2 (Pin_2), Q21.2 (D): now also D11.2 (A)
- net at J28.2 (Pin_2), Q26.2 (D): now also D12.2 (A)
- net at J27.2 (Pin_2), Q25.2 (D): now also D10.2 (A)
- net at J24.2 (Pin_2), Q22.2 (D): now also D9.2 (A)

Commit message: Fixed Schottky orientation, created 3 individual 12V pwr lines, fixed Schottky/resistor placement on layout
Connections:
- removed net +12V: D10.1 (K), D11.1 (K), D12.1 (K), D9.1 (K), J17.1 (Pin_1), J18.1 (Pin_1), J19.1 (Pin_1), J20.1 (Pin_1), J21.1 (Pin_1), J22.1 (Pin_1), J23.1 (Pin_1), J24.1 (Pin_1), J25.1 (Pin_1), J26.1 (Pin_1), J27.1 (Pin_1), J28.1 (Pin_1), J29.1 (Pin_1), J30.1 (Pin_1)
- new net +12V_FANS: D10.1 (K), D11.1 (K), D12.1 (K), D9.1 (K), J23.1 (Pin_1), J24.1 (Pin_1), J27.1 (Pin_1), J28.1 (Pin_1)
- new net +12V_HEATERS: J25.1 (Pin_1), J26.1 (Pin_1), J29.1 (Pin_1), J30.1 (Pin_1)
- new net +12V_PADS: J17.1 (Pin_1), J18.1 (Pin_1), J19.1 (Pin_1), J20.1 (Pin_1), J21.1 (Pin_1), J22.1 (Pin_1)
Changed lines of the file:
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@@
 		(in_pos_files yes)
 		(dnp no)
-		(fields_autoplaced yes)
 		(property "Reference" "#PWR076"
 			(at 44.45 36.83 0)
@@
 			)
 		)
-		(property "Value" "+12V"
-			(at 36.83 36.8299 90)
+		(property "Value" "+12V_PADS"
+			(at 34.29 34.036 90)
 			(show_name no)
 			(do_not_autoplace no)
@@
 					(size 1.27 1.27)
 				)
-				(justify left)
 			)
 		)
@@
 		(in_pos_files yes)
 		(dnp no)
-		(fields_autoplaced yes)
 		(property "Reference" "#PWR094"
 			(at 132.08 31.75 0)
@@
 			)
 		)
-		(property "Value" "+12V"
-			(at 124.46 31.7499 90)
+		(property "Value" "+12V_FANS"
+			(at 122.428 29.464 90)
 			(show_name no)
 			(do_not_autoplace no)
@@
 					(size 1.27 1.27)
 				)
-				(justify left)
 			)
 		)
@@
 		(in_pos_files yes)
 		(dnp no)
-		(fields_autoplaced yes)
 		(property "Reference" "#PWR0102"
 			(at 91.44 177.8 0)
@@
 			)
 		)
-		(property "Value" "+12V"
-			(at 83.82 177.7999 90)
+		(property "Value" "+12V_HEATERS"
+			(at 79.502 174.244 90)
 			(show_name no)
 			(do_not_autoplace no)
@@
 					(size 1.27 1.27)
 				)
-				(justify left)
 			)
 		)
@@
 		(in_pos_files yes)
 		(dnp no)
-		(fields_autoplaced yes)
 		(property "Reference" "#PWR086"
 			(at 87.63 33.02 0)
@@
 			)
 		)
-		(property "Value" "+12V"
-			(at 80.01 33.0199 90)
+		(property "Value" "+12V_PADS"
+			(at 77.724 29.972 90)
 			(show_name no)
 			(do_not_autoplace no)
@@
 					(size 1.27 1.27)
 				)
-				(justify left)
 			)
 		)
@@
 		(in_pos_files yes)
 		(dnp no)
-		(fields_autoplaced yes)
 		(property "Reference" "#PWR0103"
 			(at 175.26 35.56 0)
@@
 			)
 		)
-		(property "Value" "+12V"
-			(at 167.64 35.5599 90)
+		(property "Value" "+12V_FANS"
+			(at 165.608 33.274 90)
 			(show_name no)
 			(do_not_autoplace no)
@@
 					(size 1.27 1.27)
 				)
-				(justify left)
 			)
 		)
@@
 		(in_pos_files yes)
 		(dnp no)
-		(fields_autoplaced yes)
 		(property "Reference" "#PWR0112"
 			(at 172.72 138.43 0)
@@
 			)
 		)
-		(property "Value" "+12V"
-			(at 165.1 138.4299 90)
+		(property "Value" "+12V_HEATERS"
+			(at 161.29 134.112 90)
 			(show_name no)
 			(do_not_autoplace no)
@@
 					(size 1.27 1.27)
 				)
-				(justify left)
 			)
 		)
@@
 		(in_pos_files yes)
 		(dnp no)
-		(fields_autoplaced yes)
 		(property "Reference" "#PWR096"
 			(at 45.72 176.53 0)
@@
 			)
 		)
-		(property "Value" "+12V"
-			(at 38.1 176.5299 90)
+		(property "Value" "+12V_HEATERS"
+			(at 33.782 172.466 90)
 			(show_name no)
 			(do_not_autoplace no)
@@
 					(size 1.27 1.27)
 				)
-				(justify left)
 			)
 		)
@@
 		(in_pos_files yes)
 		(dnp no)
-		(fields_autoplaced yes)
 		(property "Reference" "#PWR093"
 			(at 129.54 76.2 0)
@@
 			)
 		)
-		(property "Value" "+12V"
-			(at 121.92 76.1999 90)
+		(property "Value" "+12V_FANS"
+			(at 119.888 73.914 90)
 			(show_name no)
 			(do_not_autoplace no)
@@
 					(size 1.27 1.27)
 				)
-				(justify left)
 			)
 		)
@@
 		(in_pos_files yes)
 		(dnp no)
-		(fields_autoplaced yes)
 		(property "Reference" "#PWR0109"
 			(at 133.35 130.81 0)
@@
 			)
 		)
-		(property "Value" "+12V"
-			(at 125.73 130.8099 90)
+		(property "Value" "+12V_HEATERS"
+			(at 121.666 127.254 90)
 			(show_name no)
 			(do_not_autoplace no)
@@
 					(size 1.27 1.27)
 				)
-				(justify left)
 			)
 		)
@@
 		(in_pos_files yes)
 		(dnp no)
-		(fields_autoplaced yes)
 		(property "Reference" "#PWR075"
 			(at 43.18 78.74 0)
@@
 			)
 		)
-		(property "Value" "+12V"
-			(at 35.56 78.7399 90)
+		(property "Value" "+12V_PADS"
+			(at 33.528 75.946 90)
 			(show_name no)
 			(do_not_autoplace no)
@@
 					(size 1.27 1.27)
 				)
-				(justify left)
 			)
 		)
@@
 		(in_pos_files yes)
 		(dnp no)
-		(fields_autoplaced yes)
 		(property "Reference" "#PWR077"
 			(at 44.45 129.54 0)
@@
 			)
 		)
-		(property "Value" "+12V"
-			(at 36.83 129.5399 90)
+		(property "Value" "+12V_PADS"
+			(at 34.29 126.238 90)
 			(show_name no)
 			(do_not_autoplace no)
@@
 					(size 1.27 1.27)
 				)
-				(justify left)
 			)
 		)
@@
 		(in_pos_files yes)
 		(dnp no)
-		(fields_autoplaced yes)
 		(property "Reference" "#PWR0104"
 			(at 175.26 90.17 0)
@@
 			)
 		)
-		(property "Value" "+12V"
-			(at 167.64 90.1699 90)
+		(property "Value" "+12V_FANS"
+			(at 165.608 88.138 90)
 			(show_name no)
 			(do_not_autoplace no)
@@
 					(size 1.27 1.27)
 				)
-				(justify left)
 			)
 		)
@@
 		(in_pos_files yes)
 		(dnp no)
-		(fields_autoplaced yes)
 		(property "Reference" "#PWR084"
 			(at 86.36 78.74 0)
@@
 			)
 		)
-		(property "Value" "+12V"
-			(at 78.74 78.7399 90)
+		(property "Value" "+12V_PADS"
+			(at 76.708 75.692 90)
 			(show_name no)
 			(do_not_autoplace no)
@@
 					(size 1.27 1.27)
 				)
-				(justify left)
 			)
 		)
@@
 		(in_pos_files yes)
 		(dnp no)
-		(fields_autoplaced yes)
 		(property "Reference" "#PWR085"
 			(at 86.36 129.54 0)
@@
 			)
 		)
-		(property "Value" "+12V"
-			(at 78.74 129.5399 90)
+		(property "Value" "+12V_PADS"
+			(at 76.708 126.238 90)
 			(show_name no)
 			(do_not_autoplace no)
@@
 					(size 1.27 1.27)
 				)
-				(justify left)
 			)
 		)
