File: usb.kicad_sch (KiCad schematic)
At the start: 12 parts, among them J1 USB_C_Receptacle_USB2.0_16P, U5 CH340C

Commit message: Fixed Schottky orientation, created 3 individual 12V pwr lines, fixed Schottky/resistor placement on layout
Connections:
- net +5V: now also D15.1 (K); no longer D15.2 (A)
- net at J1.A4 (VBUS), J1.A9 (VBUS), J1.B4 (VBUS)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: now also D15.2 (A); no longer D15.1 (K)
Changed lines of the file:
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@@
 		(lib_id "Device:D_Schottky")
 		(at 106.68 73.66 0)
+		(mirror y)
 		(unit 1)
 		(body_style 1)
@@
 		(in_pos_files yes)
 		(dnp no)
-		(fields_autoplaced yes)
 		(property "Reference" "D15"
-			(at 106.3625 67.31 0)
+			(at 106.9975 67.31 0)
 			(show_name no)
 			(do_not_autoplace no)
@@
 		)
 		(property "Value" "D_Schottky"
-			(at 106.3625 69.85 0)
+			(at 106.9975 69.85 0)
 			(show_name no)
 			(do_not_autoplace no)
